File: jantor/jantor.kicad_pcb (KiCad board)
At the start: 2 copper layers, 160.3 x 80.8 mm, 24 parts, among them K00 KEYSW, K01 KEYSW, K02 KEYSW, K03 KEYSW, K04 KEYSW, K05 KEYSW, K10 KEYSW, K11 KEYSW, K12 KEYSW, K13 KEYSW, K14 KEYSW, K15 KEYSW, K16 KEYSW, K20 KEYSW, K21 KEYSW, K22 KEYSW, K23 KEYSW, K24 KEYSW, K25 KEYSW, K30 KEYSW, K31 KEYSW, K32 KEYSW, U1 YAAJ_WeAct_BlackPill_Part_Like, U2 TRRS

Commit message: release
Parts:
- added B1: breakaway, sat1l:breakaway .75U (for 19mm net), F.Cu at (143.7, 93.8)
- added B2: breakaway, sat1l:breakaway .5U (for 19mm net), F.Cu at (143.7, 73.6)
- added B3: breakaway, sat1l:breakaway .75U (for 19mm net), F.Cu at (143.7, 53.4)
- added B4: breakaway, sat1l:breakaway .75U (for 19mm net), F.Cu at (124.7, 74.8)
- added H1: MountingHole, kbd:M2_Hole_TH_Outside, F.Cu at (162.7, 83.1)
- added H2: MountingHole, kbd:M2_Hole_TH_Outside, F.Cu at (143.7, 83.1)
- added H3: MountingHole, kbd:M2_Hole_TH_Outside, F.Cu at (219.7, 59.4)
- added H4: MountingHole, kbd:M2_Hole_TH_Outside, F.Cu at (231.6, 102.7)
- added H5: MountingHole, kbd:M2_Hole_TH_Outside, F.Cu at (143.7, 64.1)
- added H6: MountingHole, kbd:M2_Hole_TH_Outside, F.Cu at (162.7, 64.1)
Connections:
- U1 pad 37: /k01 -> unconnected-(U1-Pad37)
- U1 pad 6: unconnected-(U1-Pad6) -> /k01
- U1 pad 9: unconnected-(U1-Pad9) -> /k16
Routing:
- net /k20: track 0.00 -> 187.2 mm
- net /k10: track 0.00 -> 180.4 mm
- net /k21: track 0.00 -> 161.1 mm
- net /k00: track 0.00 -> 160.9 mm
- net /k11: track 0.00 -> 155.1 mm
- net /k22: track 0.00 -> 146.0 mm
- net /k12: track 0.00 -> 131.7 mm
- net /k23: track 0.00 -> 130.6 mm
- net /k01: track 0.00 -> 130.1 mm
- net /k24: track 0.00 -> 112.1 mm
- net /k02: track 0.00 -> 110.1 mm
- net /k13: track 0.00 -> 110.0 mm
- net /k30: track 0.00 -> 101.8 mm
- net /k14: track 0.00 -> 99.0 mm
- net +3V3: track 0.00 -> 97.4 mm
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- added copper zone on B.Cu, net GND
- added copper zone on F.Cu, net GND
Other:
- board size 160.3 x 80.8 mm -> 160.3 x 96.3 mm
