File: jantor/jantor.kicad_sch (KiCad schematic)
At the start: 34 parts, among them K00 KEYSW, K01 KEYSW, K02 KEYSW, K03 KEYSW, K04 KEYSW, K05 KEYSW, K10 KEYSW, K11 KEYSW, K12 KEYSW, K13 KEYSW, K14 KEYSW, K15 KEYSW, K16 KEYSW, K20 KEYSW, K21 KEYSW, K22 KEYSW, K23 KEYSW, K24 KEYSW, K25 KEYSW, K30 KEYSW, K31 KEYSW, K32 KEYSW, U1 YAAJ_WeAct_BlackPill_Part_Like, U2 TRRS

Commit message: what i did like whaaaa
Parts:
- added J1: Conn_01x04_Male, sat1l:Conn_01x04_Male_A, symbol Connector:Conn_01x04_Male
- added J2: Conn_01x04_Male, sat1l:Conn_01x04_Male_B, symbol Connector:Conn_01x04_Male
- added U3: YAAJ_WeAct_BlackPill_Part_Like, sat1l:Blackpill-flippy-B, symbol YAAJ_WeAct_BlackPill_Part_Like:YAAJ_WeAct_BlackPill_Part_Like
- B1, B3, B4: footprint sat1l:breakaway .75U (for 19mm net) -> sat1l:breakaway .5U (for 19mm net)
- U1: footprint Kicad-STM32:YAAJ_WeAct_BlackPill_2 -> sat1l:Blackpill-flippy-A
Connections:
- net +3V3: now also J1.1 (Pin_1), J2.1 (Pin_1), U3.20 (3V3), U3.38 (3V3)
- net GND: now also J1.4 (Pin_4), J2.4 (Pin_4), U3.19 (GND), U3.39 (GND)
- net RX: now also J1.3 (Pin_3), J2.3 (Pin_3), U3.15 (PB7)
- net TX: now also J1.2 (Pin_2), J2.2 (Pin_2), U3.14 (PB6)
- net k00: now also U1.5 (PA8), U3.5 (PA8); no longer U1.35 (PB1)
- net k01: now also U1.37 (PB10), U3.37 (PB10); no longer U1.6 (PA9)
- net k02: now also U1.4 (PB15), U3.4 (PB15); no longer U1.5 (PA8)
- net k03: now also U1.3 (PB14), U3.3 (PB14); no longer U1.4 (PB15)
- net k04: now also U1.2 (PB13), U3.2 (PB13); no longer U1.3 (PB14)
- net k05: now also U1.1 (PB12), U3.1 (PB12); no longer U1.2 (PB13)
- net k10: now also U3.17 (PB9)
- net k11: now also U3.16 (PB8)
- net k12: now also U3.13 (PB5)
- net k13: now also U1.29 (PA3), U3.29 (PA3); no longer U1.12 (PB4)
- net k14: now also U1.12 (PB4), U3.12 (PB4); no longer U1.11 (PB3)
- net k15: now also U1.11 (PB3), U3.11 (PB3); no longer U1.10 (PA15)
- net k16: now also U1.10 (PA15), U3.10 (PA15); no longer U1.9 (PA12)
- net k20: now also U1.32 (PA6), U3.32 (PA6); no longer U1.29 (PA3)
- net k21: now also U1.31 (PA5), U3.31 (PA5); no longer U1.30 (PA4)
- net k22: now also U1.30 (PA4), U3.30 (PA4); no longer U1.31 (PA5)
- net k23: now also U1.33 (PA7), U3.33 (PA7); no longer U1.32 (PA6)
- net k24: now also U1.34 (PB0), U3.34 (PB0); no longer U1.33 (PA7)
- net k25: now also U1.35 (PB1), U3.35 (PB1); no longer U1.34 (PB0)
- net k30: now also U3.28 (PA2)
- net k31: now also U3.27 (PA1)
- net k32: now also U3.26 (PA0)
- no-connect marks 12 -> 25
Other:
- moved on the sheet: U2
