File: jantor copy/jantor.kicad_sch (KiCad schematic)
At the start: 34 parts, among them K00 KEYSW, K01 KEYSW, K02 KEYSW, K03 KEYSW, K04 KEYSW, K05 KEYSW, K10 KEYSW, K11 KEYSW, K12 KEYSW, K13 KEYSW, K14 KEYSW, K15 KEYSW, K16 KEYSW, K20 KEYSW, K21 KEYSW, K22 KEYSW, K23 KEYSW, K24 KEYSW, K25 KEYSW, K30 KEYSW, K31 KEYSW, K32 KEYSW, U1 YAAJ_WeAct_BlackPill_Part_Like, U2 TRRS

Commit message: release
Parts:
- removed B1, B3, B4: breakaway, sat1l:breakaway .75U (for 19mm net), symbol Mechanical:MountingHole
- removed B2: breakaway, sat1l:breakaway .5U (for 19mm net), symbol Mechanical:MountingHole
- H1, H2, H3, H4, H5, H6: footprint kbd:M2_Hole_TH_Outside -> sat1l:M2-Plate-Hole
- K00, K01, K02, K03, K04, K05, K10, K11, K12, K13, K14, K15, K16, K20, K21, K22, K23, K24, K25, K30, K31: footprint sat1l:MXOnly-1U-Hotswap-Optional-Reversible-19mm -> sat1l:MXOnly-1U-Cutout-19mm
- K32: footprint sat1l:MXOnly-1.5U-Hotswap-Optional-Reversible-19mm -> sat1l:MXOnly-1.5U-Cutout-19mm
