File: jantor plate/jantor.kicad_pcb (KiCad board)
At the start: 2 copper layers, 153.2 x 96.3 mm, 28 parts, among them K00 KEYSW, K01 KEYSW, K02 KEYSW, K03 KEYSW, K04 KEYSW, K05 KEYSW, K10 KEYSW, K11 KEYSW, K12 KEYSW, K13 KEYSW, K14 KEYSW, K15 KEYSW, K16 KEYSW, K20 KEYSW, K21 KEYSW, K22 KEYSW, K23 KEYSW, K24 KEYSW, K25 KEYSW, K30 KEYSW, K31 KEYSW, K32 KEYSW

Commit message: а
Parts:
- removed H1, H2, H3, H4, H5, H6: MountingHole, sat1l:M2-Plate-Hole
- K00, K01, K02, K03, K04, K05, K10, K11, K12, K13, K14, K15, K16, K20, K21, K22, K23, K24, K25, K30, K31: footprint sat1l:MXOnly-1U-Cutout-19mm -> sat1l:MXOnly-1U-Cutout-LaserMargin-19mm
- K32: footprint sat1l:MXOnly-1.5U-Cutout-19mm -> sat1l:MXOnly-1.5U-Cutout-LaserMargin-19mm
- moved K00 104.6 mm to (0.00, 0.00)
- moved K01 104.6 mm to (19.0, 0.00)
- moved K02 104.6 mm to (38.0, -7.12)
- moved K03 104.6 mm to (57.0, -13.1)
- moved K04 104.6 mm to (76.0, -8.31)
- moved K05 104.6 mm to (95.0, -7.12)
- moved K10 104.6 mm to (-19.0, 20.2)
- moved K11 104.6 mm to (0.00, 19.0)
- moved K12 104.6 mm to (19.0, 19.0)
- moved K13 104.6 mm to (38.0, 11.9)
- moved K14 104.6 mm to (57.0, 5.94)
- moved K15 104.6 mm to (76.0, 10.7)
- moved K16 104.6 mm to (95.0, 11.9)
- moved K20 104.6 mm to (0.00, 38.0)
- moved K21 104.6 mm to (19.0, 38.0)
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Other:
- board size 153.2 x 96.3 mm -> 161.5 x 99.1 mm
