File: case kicad/jantor midlayer/jantor.kicad_pcb (KiCad board)
At the start: 2 copper layers, 165.5 x 99.1 mm, 0 parts

Commit message: hehehe i dont remember ANYTHING
Other:
- board size 165.5 x 99.1 mm -> 166.5 x 99.1 mm
