File: case kicad/jantor plate/jantor.kicad_pcb (KiCad board)
At the start: 2 copper layers, 161.5 x 99.1 mm, 22 parts, among them K00 KEYSW, K01 KEYSW, K02 KEYSW, K03 KEYSW, K04 KEYSW, K05 KEYSW, K10 KEYSW, K11 KEYSW, K12 KEYSW, K13 KEYSW, K14 KEYSW, K15 KEYSW, K16 KEYSW, K20 KEYSW, K21 KEYSW, K22 KEYSW, K23 KEYSW, K24 KEYSW, K25 KEYSW, K30 KEYSW, K31 KEYSW, K32 KEYSW

Commit message: hehehe i dont remember ANYTHING
Parts:
- added K00: KEYSW, sat1l:MXOnly-1U-Cutout-LaserMargin-19mm, B.Cu at (425.0, 118.6)
- added K01: KEYSW, sat1l:MXOnly-1U-Cutout-LaserMargin-19mm, B.Cu at (406.0, 118.6)
- added K02: KEYSW, sat1l:MXOnly-1U-Cutout-LaserMargin-19mm, B.Cu at (387.0, 111.5)
- added K03: KEYSW, sat1l:MXOnly-1U-Cutout-LaserMargin-19mm, B.Cu at (368.0, 105.6)
- added K04: KEYSW, sat1l:MXOnly-1U-Cutout-LaserMargin-19mm, B.Cu at (349.0, 110.3)
- added K05: KEYSW, sat1l:MXOnly-1U-Cutout-LaserMargin-19mm, B.Cu at (330.0, 111.5)
- added K10: KEYSW, sat1l:MXOnly-1U-Cutout-LaserMargin-19mm, B.Cu at (444.0, 138.8)
- added K11: KEYSW, sat1l:MXOnly-1U-Cutout-LaserMargin-19mm, B.Cu at (425.0, 137.6)
- added K12: KEYSW, sat1l:MXOnly-1U-Cutout-LaserMargin-19mm, B.Cu at (406.0, 137.6)
- added K13: KEYSW, sat1l:MXOnly-1U-Cutout-LaserMargin-19mm, B.Cu at (387.0, 130.5)
- added K14: KEYSW, sat1l:MXOnly-1U-Cutout-LaserMargin-19mm, B.Cu at (368.0, 124.6)
- added K15: KEYSW, sat1l:MXOnly-1U-Cutout-LaserMargin-19mm, B.Cu at (349.0, 129.3)
- added K16: KEYSW, sat1l:MXOnly-1U-Cutout-LaserMargin-19mm, B.Cu at (330.0, 130.5)
- added K20: KEYSW, sat1l:MXOnly-1U-Cutout-LaserMargin-19mm, B.Cu at (425.0, 156.6)
- added K21: KEYSW, sat1l:MXOnly-1U-Cutout-LaserMargin-19mm, B.Cu at (406.0, 156.6)
- added K22: KEYSW, sat1l:MXOnly-1U-Cutout-LaserMargin-19mm, B.Cu at (387.0, 149.5)
- added K23: KEYSW, sat1l:MXOnly-1U-Cutout-LaserMargin-19mm, B.Cu at (368.0, 143.6)
- added K24: KEYSW, sat1l:MXOnly-1U-Cutout-LaserMargin-19mm, B.Cu at (349.0, 148.3)
- added K25: KEYSW, sat1l:MXOnly-1U-Cutout-LaserMargin-19mm, B.Cu at (330.0, 149.5)
- added K30: KEYSW, sat1l:MXOnly-1U-Cutout-LaserMargin-19mm, B.Cu at (362.1, 167.3)
- added K31: KEYSW, sat1l:MXOnly-1U-Cutout-LaserMargin-19mm, B.Cu at (340.7, 169.7)
- added K32: KEYSW, sat1l:MXOnly-1.5U-Cutout-LaserMargin-19mm, B.Cu at (318.1, 175.0)
- moved K00 327.1 mm to (318.5, -74.4)
- moved K01 327.1 mm to (337.5, -74.4)
- moved K02 327.1 mm to (356.5, -81.6)
- moved K03 327.1 mm to (375.5, -87.5)
- moved K04 327.1 mm to (394.5, -82.8)
- moved K05 327.1 mm to (413.5, -81.6)
- moved K10 327.1 mm to (299.5, -54.2)
- moved K11 327.1 mm to (318.5, -55.4)
- moved K12 327.1 mm to (337.5, -55.4)
- moved K13 327.1 mm to (356.5, -62.6)
- moved K14 327.1 mm to (375.5, -68.5)
- moved K15 327.1 mm to (394.5, -63.8)
- moved K16 327.1 mm to (413.5, -62.6)
- moved K20 327.1 mm to (318.5, -36.4)
- moved K21 327.1 mm to (337.5, -36.4)
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Other:
- board size 161.5 x 99.1 mm -> 172 x 378.4 mm
